Commit message: 完善 TF 配置与文档，修复 pose_goal_node 阻塞问题
- ros2_control.xacro：新增7个链上关节（仅 state_interface），补全 base→L_base_link 的 TF 链
- initial_positions.yaml：追加缺失关节初始值
- real_robot.launch.py：真机 launch（仅 move_group + RViz，不含仿真组件）
- pose_goal_node.py：改为后台线程执行 plan+execute，解决 executor 阻塞
- docs/tf_configuration.md：TF 配置指南（明确区分仿真/真机）
- docs/testing_guide.md：测试步骤（启动全流程 + 测试命令）
- CLAUDE.md：追加命令行权限规则

File: src/demo/config/tianyi2_complete.ros2_control.xacro (robot description, xacro)
@@ -50,4 +50,40 @@
                 <state_interface name="velocity"/>
             </joint>
+            <!-- 以下关节仅发布状态，不参与控制，用于补全 TF 链 -->
+            <joint name="left_tcp_joint">
+                <state_interface name="position">
+                  <param name="initial_value">0.0</param>
+                </state_interface>
+            </joint>
+            <joint name="left_hand_to_tcp">
+                <state_interface name="position">
+                  <param name="initial_value">0.0</param>
+                </state_interface>
+            </joint>
+            <joint name="shoulder_pitch_l_joint">
+                <state_interface name="position">
+                  <param name="initial_value">0.0</param>
+                </state_interface>
+            </joint>
+            <joint name="waist_yaw_joint">
+                <state_interface name="position">
+                  <param name="initial_value">0.0</param>
+                </state_interface>
+            </joint>
+            <joint name="waist_pitch_joint">
+                <state_interface name="position">
+                  <param name="initial_value">0.0</param>
+                </state_interface>
+            </joint>
+            <joint name="second_leg_pitch_joint">
+                <state_interface name="position">
+                  <param name="initial_value">0.0</param>
+                </state_interface>
+            </joint>
+            <joint name="first_leg_pitch_joint">
+                <state_interface name="position">
+                  <param name="initial_value">0.0</param>
+                </state_interface>
+            </joint>
         </ros2_control>
     </xacro:macro>

Commit message: 重构：双臂规划组(L_Arm_Group+R_Arm_group)，4话题控制节点，补全TF链
- SRDF: 新增 R_Arm_group，重命名 hand_L_Arn_Group → L_Arm_Group
- pose_goal_node: 解耦为 /left_arm + /right_arm 各两话题 (target_pose + delta_pose)
- ros2_control.xacro: 追加6个被动关节补全TF链 (first_leg~shoulder_pitch)
- 更新 CLAUDE.md、testing_guide.md、tf_configuration.md 等所有文档

File: src/demo/config/tianyi2_complete.ros2_control.xacro (robot description, xacro)
@@ -50,38 +50,75 @@
                 <state_interface name="velocity"/>
             </joint>
-            <!-- 以下关节仅发布状态，不参与控制，用于补全 TF 链 -->
-            <joint name="left_tcp_joint">
+            <joint name="shoulder_roll_r_joint">
+                <command_interface name="position"/>
                 <state_interface name="position">
-                  <param name="initial_value">0.0</param>
+                  <param name="initial_value">${initial_positions['shoulder_roll_r_joint']}</param>
+                </state_interface>
+                <state_interface name="velocity"/>
+            </joint>
+            <joint name="shoulder_yaw_r_joint">
+                <command_interface name="position"/>
+                <state_interface name="position">
+                  <param name="initial_value">${initial_positions['shoulder_yaw_r_joint']}</param>
+                </state_interface>
+                <state_interface name="velocity"/>
+            </joint>
+            <joint name="elbow_pitch_r_joint">
+                <command_interface name="position"/>
+                <state_interface name="position">
+                  <param name="initial_value">${initial_positions['elbow_pitch_r_joint']}</param>
+                </state_interface>
+                <state_interface name="velocity"/>
+            </joint>
+            <joint name="elbow_yaw_r_joint">
+                <command_interface name="position"/>
+                <state_interface name="position">
+                  <param name="initial_value">${initial_positions['elbow_yaw_r_joint']}</param>
+                </state_interface>
+                <state_interface name="velocity"/>
+            </joint>
+            <joint name="wrist_pitch_r_joint">
+                <command_interface name="position"/>
+                <state_interface name="position">
+                  <param name="initial_value">${initial_positions['wrist_pitch_r_joint']}</param>
+                </state_interface>
+                <state_interface name="velocity"/>
+            </joint>
+            <joint name="wrist_roll_r_joint">
+                <command_interface name="position"/>
+                <state_interface name="position">
+                  <param name="initial_value">${initial_positions['wrist_roll_r_joint']}</param>
+                </state_interface>
+                <state_interface name="velocity"/>
+            </joint>
+            <!-- 仅上报状态（不参与控制），补全 TF 链 -->
+            <joint name="shoulder_pitch_l_joint">
+                <state_interface name="position">
+                  <param name="initial_value">${initial_positions['shoulder_pitch_l_joint']}</param>
                 </state_interface>
             </joint>
-            <joint name="left_hand_to_tcp">
+            <joint name="shoulder_pitch_r_joint">
                 <state_interface name="position">
-                  <param name="initial_value">0.0</param>
-                </state_interface>
-            </joint>
-            <joint name="shoulder_pitch_l_joint">
-                <state_interface name="position">
-                  <param name="initial_value">0.0</param>
+                  <param name="initial_value">${initial_positions['shoulder_pitch_r_joint']}</param>
                 </state_interface>
             </joint>
             <joint name="waist_yaw_joint">
                 <state_interface name="position">
-                  <param name="initial_value">0.0</param>
+                  <param name="initial_value">${initial_positions['waist_yaw_joint']}</param>
                 </state_interface>
             </joint>
             <joint name="waist_pitch_joint">
                 <state_interface name="position">
-                  <param name="initial_value">0.0</param>
+                  <param name="initial_value">${initial_positions['waist_pitch_joint']}</param>
                 </state_interface>
             </joint>
             <joint name="second_leg_pitch_joint">
                 <state_interface name="position">
-                  <param name="initial_value">0.0</param>
+                  <param name="initial_value">${initial_positions['second_leg_pitch_joint']}</param>
                 </state_interface>
             </joint>
             <joint name="first_leg_pitch_joint">
                 <state_interface name="position">
-                  <param name="initial_value">0.0</param>
+                  <param name="initial_value">${initial_positions['first_leg_pitch_joint']}</param>
                 </state_interface>
             </joint>
