Commit message: fix: 补全 L_Arm 控制器 action_ns，统一命名，补 TF 躯干被动关节
- moveit_controllers.yaml: L_Arm_Group_controller 补上缺失的 action_ns 和 default
- 统一命名: R_Arm_group_controller → R_Arm_Group_controller
- ros2_control.xacro: 新增 first_leg_pitch/second_leg_pitch/waist_pitch/waist_yaw 关节（仅 state_interface）
- initial_positions.yaml: 补上对应躯干关节初始值
- MoveIt 配置从 demo/ 迁移至 tianyi2_moveit/
- 新增 bridge_node.py 及 motor_config.yaml

Co-Authored-By: Claude <noreply@anthropic.com>

File: src/tianyi2_moveit/config/tianyi2_complete.ros2_control.xacro (robot description, xacro)
@@ -8,4 +8,11 @@
                 <plugin>mock_components/GenericSystem</plugin>
             </hardware>
+            <joint name="shoulder_pitch_l_joint">
+                <command_interface name="position"/>
+                <state_interface name="position">
+                  <param name="initial_value">${initial_positions['shoulder_pitch_l_joint']}</param>
+                </state_interface>
+                <state_interface name="velocity"/>
+            </joint>
             <joint name="shoulder_roll_l_joint">
                 <command_interface name="position"/>
@@ -47,4 +54,11 @@
                 <state_interface name="position">
                   <param name="initial_value">${initial_positions['wrist_roll_l_joint']}</param>
+                </state_interface>
+                <state_interface name="velocity"/>
+            </joint>
+            <joint name="shoulder_pitch_r_joint">
+                <command_interface name="position"/>
+                <state_interface name="position">
+                  <param name="initial_value">${initial_positions['shoulder_pitch_r_joint']}</param>
                 </state_interface>
                 <state_interface name="velocity"/>
@@ -92,14 +106,22 @@
                 <state_interface name="velocity"/>
             </joint>
-            <!-- 仅上报状态（不参与控制），补全 TF 链 -->
-            <joint name="shoulder_pitch_l_joint">
+            <!-- 仅发布状态，不参与控制（补全 base→手臂 的 TF 链） -->
+            <joint name="first_leg_pitch_joint">
                 <state_interface name="position">
-                  <param name="initial_value">${initial_positions['shoulder_pitch_l_joint']}</param>
+                  <param name="initial_value">${initial_positions['first_leg_pitch_joint']}</param>
                 </state_interface>
+                <state_interface name="velocity"/>
             </joint>
-            <joint name="shoulder_pitch_r_joint">
+            <joint name="second_leg_pitch_joint">
                 <state_interface name="position">
-                  <param name="initial_value">${initial_positions['shoulder_pitch_r_joint']}</param>
+                  <param name="initial_value">${initial_positions['second_leg_pitch_joint']}</param>
                 </state_interface>
+                <state_interface name="velocity"/>
+            </joint>
+            <joint name="waist_pitch_joint">
+                <state_interface name="position">
+                  <param name="initial_value">${initial_positions['waist_pitch_joint']}</param>
+                </state_interface>
+                <state_interface name="velocity"/>
             </joint>
             <joint name="waist_yaw_joint">
@@ -107,19 +129,5 @@
                   <param name="initial_value">${initial_positions['waist_yaw_joint']}</param>
                 </state_interface>
-            </joint>
-            <joint name="waist_pitch_joint">
-                <state_interface name="position">
-                  <param name="initial_value">${initial_positions['waist_pitch_joint']}</param>
-                </state_interface>
-            </joint>
-            <joint name="second_leg_pitch_joint">
-                <state_interface name="position">
-                  <param name="initial_value">${initial_positions['second_leg_pitch_joint']}</param>
-                </state_interface>
-            </joint>
-            <joint name="first_leg_pitch_joint">
-                <state_interface name="position">
-                  <param name="initial_value">${initial_positions['first_leg_pitch_joint']}</param>
-                </state_interface>
+                <state_interface name="velocity"/>
             </joint>
         </ros2_control>
